Commit message: i was using both the source and binary installation of the ros2 universal robots driver, now only the iron binary installtion.

File: src/my_robot_cell/my_robot_cell_control/urdf/my_robot_cell_controlled.urdf.xacro (robot description, xacro)
@@ -3,43 +3,84 @@
   <!--First, include the macro from our custom description-->
   <xacro:include filename="$(find my_robot_cell_description)/urdf/my_robot_cell_macro.xacro"/>
-  <!--The driver already provides a control tag for the UR arm, we can directly include-->
-  <xacro:include filename="$(find ur_description)/urdf/ur.ros2_control.xacro"/>
-  <!--We need to specify the arguments used for parametrizing our description-->
+  <!-- robot name parameter -->
+  <xacro:arg name="name" default="ur"/>
+  <!-- possible 'ur_type' values: ur3, ur3e, ur5, ur5e, ur10, ur10e, ur16e, ur20, ur30 -->
   <xacro:arg name="ur_type" default="ur5e"/>
-  <xacro:arg name="joint_limit_parameters_file" default="$(find ur_description)/config/$(arg ur_type)/joint_limits.yaml"/>
+  <xacro:arg name="tf_prefix" default="" />
+  <xacro:arg name="joint_limits_parameters_file" default="$(find ur_description)/config/$(arg ur_type)/joint_limits.yaml"/>
   <xacro:arg name="kinematics_parameters_file" default="$(find ur_description)/config/$(arg ur_type)/default_kinematics.yaml"/>
   <xacro:arg name="physical_parameters_file" default="$(find ur_description)/config/$(arg ur_type)/physical_parameters.yaml"/>
   <xacro:arg name="visual_parameters_file" default="$(find ur_description)/config/$(arg ur_type)/visual_parameters.yaml"/>
-  <xacro:arg name="robot_ip" default="10.130.1.100"/>
+  <xacro:arg name="transmission_hw_interface" default=""/>
+  <xacro:arg name="safety_limits" default="false"/>
+  <xacro:arg name="safety_pos_margin" default="0.15"/>
+  <xacro:arg name="safety_k_position" default="20"/>
   <xacro:arg name="headless_mode" default="false" />
-  <xacro:arg name="ur_script_filename" default="$(find ur_client_library)/resources/external_control.urscript"/>
-  <xacro:arg name="ur_output_recipe_filename" default="$(find ur_robot_driver)/resources/rtde_output_recipe.txt"/>
-  <xacro:arg name="ur_input_recipe_filename" default="$(find ur_robot_driver)/resources/rtde_input_recipe.txt"/>
-  <xacro:arg name="use_mock_hardware" default="false" />
-  <xacro:arg name="mock_sensor_commands" default="false" />
-  <xacro:arg name="hash_kinematics" default="calib_2089462667388424822"/>
-  <link name="world" />
+  <xacro:arg name="robot_ip" default="10.130.1.100" />
+  <xacro:arg name="script_filename" default=""/>
+  <xacro:arg name="output_recipe_filename" default=""/>
+  <xacro:arg name="input_recipe_filename" default=""/>
+  <xacro:arg name="reverse_ip" default="0.0.0.0"/>
+  <xacro:arg name="script_command_port" default="50004"/>
+  <xacro:arg name="reverse_port" default="50001"/>
+  <xacro:arg name="script_sender_port" default="50002"/>
+  <xacro:arg name="trajectory_port" default="50003"/>
+  <!-- Tool communication related parameters -->
+  <xacro:arg name="use_tool_communication" default="false" />
+  <xacro:arg name="tool_voltage" default="0" />
+  <xacro:arg name="tool_parity" default="0" />
+  <xacro:arg name="tool_baud_rate" default="115200" />
+  <xacro:arg name="tool_stop_bits" default="1" />
+  <xacro:arg name="tool_rx_idle_chars" default="1.5" />
+  <xacro:arg name="tool_tx_idle_chars" default="3.5" />
+  <xacro:arg name="tool_device_name" default="/tmp/ttyUR" />
+  <xacro:arg name="tool_tcp_port" default="54321" />
+  <!-- Simulation parameters -->
+  <xacro:arg name="use_fake_hardware" default="false" />
+  <xacro:arg name="fake_sensor_commands" default="false" />
+  <xacro:arg name="sim_ignition" default="false" />
+  <xacro:arg name="simulation_controllers" default="" />
+  <!-- initial position for simulations (Fake Hardware, Ignition) -->
+  <xacro:arg name="initial_positions_file" default="$(find ur_description)/config/initial_positions.yaml"/>
+  <xacro:property name="initial_positions_file" default="$(arg initial_positions_file)"/>
+  <link name="world"/>
   <!--Create the scene description including the robot-->
-  <xacro:my_robot_cell
+<xacro:my_robot_cell
     parent="world"
     ur_type="$(arg ur_type)"
-    joint_limits_parameters_file="$(arg joint_limit_parameters_file)"
+    joint_limits_parameters_file="$(arg joint_limits_parameters_file)"
     kinematics_parameters_file="$(arg kinematics_parameters_file)"
     physical_parameters_file="$(arg physical_parameters_file)"
     visual_parameters_file="$(arg visual_parameters_file)"
-  >
-    <origin xyz="0 0 1" rpy="0 0 0" />
+    transmission_hw_interface="$(arg transmission_hw_interface)"
+    safety_limits="$(arg safety_limits)"
+    safety_pos_margin="$(arg safety_pos_margin)"
+    safety_k_position="$(arg safety_k_position)"
+    use_fake_hardware="$(arg use_fake_hardware)"
+    fake_sensor_commands="$(arg fake_sensor_commands)"
+    sim_ignition="$(arg sim_ignition)"
+    headless_mode="$(arg headless_mode)"
+    initial_positions="${xacro.load_yaml(initial_positions_file)}"
+    use_tool_communication="$(arg use_tool_communication)"
+    tool_voltage="$(arg tool_voltage)"
+    tool_parity="$(arg tool_parity)"
+    tool_baud_rate="$(arg tool_baud_rate)"
+    tool_stop_bits="$(arg tool_stop_bits)"
+    tool_rx_idle_chars="$(arg tool_rx_idle_chars)"
+    tool_tx_idle_chars="$(arg tool_tx_idle_chars)"
+    tool_device_name="$(arg tool_device_name)"
+    tool_tcp_port="$(arg tool_tcp_port)"
+    robot_ip="$(arg robot_ip)"
+    script_filename="$(arg script_filename)"
+    output_recipe_filename="$(arg output_recipe_filename)"
+    input_recipe_filename="$(arg input_recipe_filename)"
+    reverse_ip="$(arg reverse_ip)"
+    script_command_port="$(arg script_command_port)"
+    reverse_port="$(arg reverse_port)"
+    script_sender_port="$(arg script_sender_port)"
+    trajectory_port="$(arg trajectory_port)"
+    >
+      <origin xyz="0 0 1" rpy="0 0 0" />
   </xacro:my_robot_cell>
-  <!--Create the control tag for the UR robot-->
-  <xacro:ur_ros2_control
-    name="$(arg ur_type)"
-    tf_prefix="$(arg ur_type)_"
-    robot_ip="$(arg robot_ip)"
-    script_filename="$(arg ur_script_filename)"
-    output_recipe_filename="$(arg ur_output_recipe_filename)"
-    input_recipe_filename="$(arg ur_input_recipe_filename)"
-    headless_mode="$(arg headless_mode)"
-    hash_kinematics="$arg hash_kinematics"
-  />
   <!--If you had more controlled devices in your description, e.g. a gripper, you can add another ros2_control tag here-->
 </robot>

File: src/my_robot_cell/my_robot_cell_description/urdf/my_robot_cell.urdf.xacro (robot description, xacro)
@@ -1,12 +1,48 @@
 <?xml version="1.0"?>
 <robot name="my_robot_cell" xmlns:xacro="http://ros.org/wiki/xacro">
+  <!-- First, include the macro from our custom description -->
   <xacro:include filename="$(find my_robot_cell_description)/urdf/my_robot_cell_macro.xacro"/>
+  <!-- Robot name parameter -->
+  <xacro:arg name="name" default="ur"/>
   <xacro:arg name="ur_type" default="ur5e"/>
+  <xacro:arg name="tf_prefix" default="" />
   <xacro:arg name="joint_limits_parameters_file" default="$(find ur_description)/config/$(arg ur_type)/joint_limits.yaml"/>
   <xacro:arg name="kinematics_parameters_file" default="$(find ur_description)/config/$(arg ur_type)/default_kinematics.yaml"/>
   <xacro:arg name="physical_parameters_file" default="$(find ur_description)/config/$(arg ur_type)/physical_parameters.yaml"/>
   <xacro:arg name="visual_parameters_file" default="$(find ur_description)/config/$(arg ur_type)/visual_parameters.yaml"/>
+  <xacro:arg name="transmission_hw_interface" default=""/>
+  <xacro:arg name="safety_limits" default="false"/>
+  <xacro:arg name="safety_pos_margin" default="0.15"/>
+  <xacro:arg name="safety_k_position" default="20"/>
+  <xacro:arg name="headless_mode" default="false" />
+  <xacro:arg name="robot_ip" default="10.130.1.100" />
+  <xacro:arg name="script_filename" default=""/>
+  <xacro:arg name="output_recipe_filename" default=""/>
+  <xacro:arg name="input_recipe_filename" default=""/>
+  <xacro:arg name="reverse_ip" default="0.0.0.0"/>
+  <xacro:arg name="script_command_port" default="50004"/>
+  <xacro:arg name="reverse_port" default="50001"/>
+  <xacro:arg name="script_sender_port" default="50002"/>
+  <xacro:arg name="trajectory_port" default="50003"/>
+  <!-- Tool communication related parameters -->
+  <xacro:arg name="use_tool_communication" default="false" />
+  <xacro:arg name="tool_voltage" default="0" />
+  <xacro:arg name="tool_parity" default="0" />
+  <xacro:arg name="tool_baud_rate" default="115200" />
+  <xacro:arg name="tool_stop_bits" default="1" />
+  <xacro:arg name="tool_rx_idle_chars" default="1.5" />
+  <xacro:arg name="tool_tx_idle_chars" default="3.5" />
+  <xacro:arg name="tool_device_name" default="/tmp/ttyUR" />
+  <xacro:arg name="tool_tcp_port" default="54321" />
+  <!-- Simulation parameters -->
+  <xacro:arg name="use_fake_hardware" default="false" />
+  <xacro:arg name="fake_sensor_commands" default="false" />
+  <xacro:arg name="sim_ignition" default="false" />
+  <xacro:arg name="simulation_controllers" default="" />
+  <!-- Initial position for simulations (Fake Hardware, Ignition) -->
+  <xacro:arg name="initial_positions_file" default="$(find ur_description)/config/initial_positions.yaml"/>
+  <xacro:property name="initial_positions_file" default="$(arg initial_positions_file)"/>
   <link name="world"/>
-  <!--This will create the scene where the robot is located in-->
+  <!-- Create the scene description including the robot -->
   <xacro:my_robot_cell
     parent="world"
@@ -16,4 +52,31 @@
     physical_parameters_file="$(arg physical_parameters_file)"
     visual_parameters_file="$(arg visual_parameters_file)"
+    transmission_hw_interface="$(arg transmission_hw_interface)"
+    safety_limits="$(arg safety_limits)"
+    safety_pos_margin="$(arg safety_pos_margin)"
+    safety_k_position="$(arg safety_k_position)"
+    use_fake_hardware="$(arg use_fake_hardware)"
+    fake_sensor_commands="$(arg fake_sensor_commands)"
+    sim_ignition="$(arg sim_ignition)"
+    headless_mode="$(arg headless_mode)"
+    initial_positions="${xacro.load_yaml(initial_positions_file)}"
+    use_tool_communication="$(arg use_tool_communication)"
+    tool_voltage="$(arg tool_voltage)"
+    tool_parity="$(arg tool_parity)"
+    tool_baud_rate="$(arg tool_baud_rate)"
+    tool_stop_bits="$(arg tool_stop_bits)"
+    tool_rx_idle_chars="$(arg tool_rx_idle_chars)"
+    tool_tx_idle_chars="$(arg tool_tx_idle_chars)"
+    tool_device_name="$(arg tool_device_name)"
+    tool_tcp_port="$(arg tool_tcp_port)"
+    robot_ip="$(arg robot_ip)"
+    script_filename="$(arg script_filename)"
+    output_recipe_filename="$(arg output_recipe_filename)"
+    input_recipe_filename="$(arg input_recipe_filename)"
+    reverse_ip="$(arg reverse_ip)"
+    script_command_port="$(arg script_command_port)"
+    reverse_port="$(arg reverse_port)"
+    script_sender_port="$(arg script_sender_port)"
+    trajectory_port="$(arg trajectory_port)"
     >
       <origin xyz="0 0 1" rpy="0 0 0" />

File: src/my_robot_cell/my_robot_cell_description/urdf/my_robot_cell_macro.xacro (robot description, xacro)
@@ -10,5 +10,33 @@
     physical_parameters_file
     visual_parameters_file
+    transmission_hw_interface
+    safety_limits
+    safety_pos_margin
+    safety_k_position
+    use_fake_hardware
+    fake_sensor_commands
+    sim_ignition
+    headless_mode
+    initial_positions
+    use_tool_communication
+    tool_voltage
+    tool_parity
+    tool_baud_rate
+    tool_stop_bits
+    tool_rx_idle_chars
+    tool_tx_idle_chars
+    tool_device_name
+    tool_tcp_port
+    robot_ip
+    script_filename
+    output_recipe_filename
+    input_recipe_filename
+    reverse_ip
+    script_command_port
+    reverse_port
+    script_sender_port
+    trajectory_port
     ">
+    <!-- Joint connecting the table to the parent link -->
     <joint name="table_base_joint" type="fixed">
       <xacro:insert_block name="origin" />
@@ -16,4 +44,5 @@
       <child link="table" />
     </joint>
+    <!-- Definition of the table link with visual and collision geometry -->
     <link name="table">
       <visual>
@@ -30,4 +59,5 @@
       </collision>
     </link>
+    <!-- Definition of the monitor link with visual and collision geometry -->
     <link name="monitor">
       <visual>
@@ -42,4 +72,5 @@
       </collision>
     </link>
+    <!-- Joint connecting the monitor to the table -->
     <joint name="base_to_monitor" type="fixed">
       <parent link="table"/>
@@ -47,7 +78,9 @@
       <origin xyz="0.2 0.6 0"/>
     </joint>
+    <!-- Material definition (not currently used, but defined for potential future use) -->
     <material name="white">
       <color rgba="1 1 1 1"/>
     </material>
+    <!-- Definition of the wall link with visual and collision geometry -->
     <link name="wall">
       <visual>
@@ -62,4 +95,5 @@
       </collision>
     </link>
+    <!-- Joint connecting the wall to the table -->
     <joint name="base_to_wall" type="fixed">
       <parent link="table"/>
@@ -67,5 +101,7 @@
       <origin xyz="1.25 1.5 0.5"/>
     </joint>
+    <!-- Definition of the robot mount link -->
     <link name="robot_mount"/>
+    <!-- Joint connecting the robot mount to the table -->
     <joint name="base_to_robot_mount" type="fixed">
       <parent link="table"/>
@@ -73,5 +109,5 @@
       <origin xyz="0.845 0.85 0" rpy="0 0 ${pi}" />
     </joint>
-    <!--This will create the specific robot-->
+    <!-- Instantiate the robot using the URDF macro -->
     <xacro:ur_robot
       name="${ur_type}"
@@ -82,4 +118,31 @@
       physical_parameters_file="${physical_parameters_file}"
       visual_parameters_file="${visual_parameters_file}"
+      transmission_hw_interface="${transmission_hw_interface}"
+      safety_limits="${safety_limits}"
+      safety_pos_margin="${safety_pos_margin}"
+      safety_k_position="${safety_k_position}"
+      use_fake_hardware="${use_fake_hardware}"
+      fake_sensor_commands="${fake_sensor_commands}"
+      sim_ignition="${sim_ignition}"
+      headless_mode="${headless_mode}"
+      initial_positions="${initial_positions}"
+      use_tool_communication="${use_tool_communication}"
+      tool_voltage="${tool_voltage}"
+      tool_parity="${tool_parity}"
+      tool_baud_rate="${tool_baud_rate}"
+      tool_stop_bits="${tool_stop_bits}"
+      tool_rx_idle_chars="${tool_rx_idle_chars}"
+      tool_tx_idle_chars="${tool_tx_idle_chars}"
+      tool_device_name="${tool_device_name}"
+      tool_tcp_port="${tool_tcp_port}"
+      robot_ip="${robot_ip}"
+      script_filename="${script_filename}"
+      output_recipe_filename="${output_recipe_filename}"
+      input_recipe_filename="${input_recipe_filename}"
+      reverse_ip="${reverse_ip}"
+      script_command_port="${script_command_port}"
+      reverse_port="${reverse_port}"
+      script_sender_port="${script_sender_port}"
+      trajectory_port="${trajectory_port}"
     >
       <origin xyz="0 0 0" rpy="0 0 0" />
